File: hardware/EEG_Kicad_Project/usb.kicad_sch (KiCad schematic)
At the start: 0 parts

Commit message: added 3V3 /-2V5 wiring on schematic
Other:
- note added: "USB C"
Changed lines of the file:
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@@
 	(generator_version "9.0")
 	(paper "A4")
+	(text "USB C"
+		(exclude_from_sim no)
+		(at 41.656 23.114 0)
+		(effects
+			(font
+				(size 2.54 2.54)
+				(thickness 0.508)
+				(bold yes)
+				(color 0 0 194 1)
+			)
+		)
+	)
 )
