File: hardware/EEG_Kicad_Project/stm32.kicad_sch (KiCad schematic)
At the start: 14 parts, among them SW1 SW_Push, U1 STM32F446RETx

Commit message: Add USB galvanic isolation barrier for patient safety
Adds a USB-C receptacle -> ESD protection -> ADuM3160 isolator ->
isolated TMU3-0511 DC-DC chain, separating the STM32/ADS1299/analog
supply (now fully isolated) from the non-isolated USB-connector side.
Closes the previously-floating USB_OTG_FS_DP/DM pins on the STM32,
adds CC1/CC2 pulldowns and VBUS decoupling on the new receptacle, and
fixes ADuM3160 VBUS2 tie per datasheet. Verified via kicad-happy: no
ERC regressions, isolation barrier confirmed intact (no net bridges
GND_PRI/+5V_PRI with the isolated GNDA/+5V/+3V3 domain).

Co-Authored-By: Claude Sonnet 5 <noreply@anthropic.com>
Changed lines of the file:
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@@
 	(wire
 		(pts
-			(xy 180.34 88.9) (xy 182.88 88.9)
+			(xy 180.34 88.9) (xy 199.39 88.9)
 		)
 		(stroke
@@
 	(wire
 		(pts
+			(xy 199.39 88.9) (xy 199.39 87.63)
+		)
+		(stroke
+			(width 0)
+			(type default)
+		)
+	)
+	(wire
+		(pts
 			(xy 31.75 40.64) (xy 31.75 44.45)
 		)
@@
 	(wire
 		(pts
-			(xy 180.34 91.44) (xy 182.88 91.44)
+			(xy 180.34 91.44) (xy 203.2 91.44)
 		)
 		(stroke
@@
 	(wire
 		(pts
+			(xy 203.2 91.44) (xy 203.2 87.63)
+		)
+		(stroke
+			(width 0)
+			(type default)
+		)
+	)
+	(wire
+		(pts
 			(xy 43.18 40.64) (xy 43.18 44.45)
 		)
@@
 			(width 0)
 			(type default)
-		)
-	)
-	(label "USB_OTG_FS_DP"
-		(at 182.88 91.44 0)
-		(effects
-			(font
-				(size 1.27 1.27)
-			)
-			(justify left bottom)
 		)
 	)
@@
 		)
 	)
-	(label "USB_OTG_FS_DM"
-		(at 182.88 88.9 0)
-		(effects
-			(font
-				(size 1.27 1.27)
-			)
-			(justify left bottom)
-		)
-	)
 	(label "RCC_OSC_OUT"
 		(at 135.89 73.66 180)
@@
 		)
 	)
+	(global_label "USB_OTG_FS_DP"
+		(shape input)
+		(at 203.2 87.63 90)
+		(fields_autoplaced yes)
+		(effects
+			(font
+				(size 1.27 1.27)
+			)
+			(justify left)
+		)
+		(property "Intersheetrefs" "${INTERSHEET_REFS}"
+			(at 203.2 69.5258 90)
+			(effects
+				(font
+					(size 1.27 1.27)
+				)
+				(justify left)
+				(hide yes)
+			)
+		)
+	)
+	(global_label "USB_OTG_FS_DM"
+		(shape input)
+		(at 199.39 87.63 90)
+		(fields_autoplaced yes)
+		(effects
+			(font
+				(size 1.27 1.27)
+			)
+			(justify left)
+		)
+		(property "Intersheetrefs" "${INTERSHEET_REFS}"
+			(at 199.39 69.3444 90)
+			(effects
+				(font
+					(size 1.27 1.27)
+				)
+				(justify left)
+				(hide yes)
+			)
+		)
+	)
